Commit message: add another cylinder with joint

File: urdf/my_robot.urdf (robot description, URDF)
Before this commit: robot my_robot, 1 links, 0 joints
Links:
- added link second_link; visual cylinder length=0.2 radius=0.1
Joints:
- added joint base_second_joint: type fixed, parent base_link, child second_link, origin xyz=0 0 0 rpy=0 0 0

Commit message: fix joint position and object placement position

File: urdf/my_robot.urdf (robot description, URDF)
Before this commit: robot my_robot, 2 links, 1 joints
Joints:
- joint base_second_joint: origin xyz=0 0 0 rpy=0 0 0 -> xyz=0 0 0.2 rpy=0 0 0

Commit message: joint type
try revolute

File: urdf/my_robot.urdf (robot description, URDF)
Before this commit: robot my_robot, 3 links, 2 joints
Links:
- removed link third_link
Joints:
- removed joint second_third_joint
- joint base_second_joint: axis (none) -> 0 0 1; limit (none) -> lower=-1.57 upper=1.57 effort=100 velocity=100; type fixed -> revolute

Commit message: prismatic

File: urdf/my_robot.urdf (robot description, URDF)
Before this commit: robot my_robot, 2 links, 1 joints
Joints:
- joint base_second_joint: axis 0 0 1 -> 1 0 0; limit lower=-1.57 upper=1.57 effort=100 velocity=100 -> lower=0.0 upper=0.2 effort=100 velocity=100; type revolute -> prismatic

Commit message: right and left wheels with joint

File: urdf/my_robot.urdf (robot description, URDF)
Before this commit: robot my_robot, 2 links, 1 joints
Links:
- removed link second_link
- added link left_wheel_link; visual cylinder length=0.05 radius=0.1
- added link right_wheel_link; visual cylinder length=0.05 radius=0.1
Joints:
- removed joint base_second_joint
- added joint base_left_wheel_joint: type continuous, parent base_link, child left_wheel_link, origin xyz=-0.15 0.225 0 rpy=0 0 0, axis 0 1 0
- added joint base_right_wheel_joint: type continuous, parent base_link, child right_wheel_link, origin xyz=-0.15 -0.225 0 rpy=0 0 0, axis 0 1 0

Commit message: Revert "right and left wheels with joint"
This reverts commit 6ed44cfcc5b67a2e87ec68c30bd8c84d6f530fd1.

File: urdf/my_robot.urdf (robot description, URDF)
Before this commit: robot my_robot, 3 links, 2 joints
Links:
- removed link left_wheel_link
- removed link right_wheel_link
- added link second_link; visual cylinder length=0.2 radius=0.1
Joints:
- removed joint base_left_wheel_joint
- removed joint base_right_wheel_joint
- added joint base_second_joint: type prismatic, parent base_link, child second_link, origin xyz=0 0 0.2 rpy=0 0 0, axis 1 0 0, limit lower=0.0 upper=0.2 effort=100 velocity=100

Commit message: Add cater wheel

File: urdf/my_robot.urdf (robot description, URDF)
Before this commit: robot my_robot, 3 links, 2 joints
Links:
- added link caster_wheel_link; visual sphere radius=0.05
Joints:
- added joint base_caster_wheel_joint: type fixed, parent base_link, child caster_wheel_link, origin xyz=0.2 0 -0.05 rpy=0 0 0, axis 0 0 0
