Commit message: gazebo camera frame is inconsistent with rviz + opencv convention

File: ros2_ws/src/my_robot_description/urdf/camera.xacro (robot description, xacro)
@@ -24,4 +24,13 @@
         <origin xyz="${base_length/2 + camera_length/2.0} 0 ${base_height/2}" rpy="0 0 0" />
     </joint>
+    <link name="camera_link_optical" />
+    <joint name="camera_optical_joint" type="fixed">
+        <!-- these values have to be these values otherwise the gazebo camera
+            image won't be aligned properly with the frame it is supposedly
+            originating from -->
+        <origin xyz="0 0 0" rpy="${-pi/2} 0 ${-pi/2}"/>
+        <parent link="camera_link"/>
+        <child link="camera_link_optical"/>
+    </joint>
     <gazebo reference="camera_link">
         <sensor name="camera" type="camera">
@@ -42,5 +51,5 @@
                     <stddev>0.007</stddev>
                 </noise>
-                <optical_frame_id>camera_link</optical_frame_id>
+                <optical_frame_id>camera_link_optical</optical_frame_id>
                 <camera_info_topic>camera/camera_info</camera_info_topic>
             </camera>
