Commit message: Add inertial tags in the urdf

File: ros2_ws/src/my_robot_description/urdf/common_properties.xacro (robot description, xacro)
@@ -7,3 +7,12 @@
         <color rgba="0.5 0.5 0.5 1" />
     </material>
+    <xacro:macro name="box_intertia" params="m x y z o_xyz o_rpy">
+        <inertial>
+            <mass value="${m}" />
+            <origin xyz="${o_xyz}" rpy="${o_rpy}" />
+            <inertial ixx="${(m/12) * (y*y + z*z)}" ixy="0" ixz="0"
+                      iyy="${(m/12) * (x*x + z*z)}" iyz="0"
+                      izz="${(m/12) * (x*x + y*y)}" />
+        </inertial>
+    </xacro:macro>
 </robot>

File: ros2_ws/src/my_robot_description/urdf/mobile_base.xacro (robot description, xacro)
@@ -15,4 +15,6 @@
             <material name="blue" />
         </visual>
+        <xacro:box_intertia m="5.0" x="${base_length}" y="${base_width}" z="${base_height}"
+                            o_xyz="0 0 ${base_height / 2.0}" o_rpy="0 0 0" />
     </link>
     <xacro:macro name="wheel_link" params="prefix">

Commit message: Fix inertia

File: ros2_ws/src/my_robot_description/urdf/common_properties.xacro (robot description, xacro)
@@ -7,11 +7,11 @@
         <color rgba="0.5 0.5 0.5 1" />
     </material>
-    <xacro:macro name="box_intertia" params="m x y z o_xyz o_rpy">
+    <xacro:macro name="box_inertia" params="m x y z o_xyz o_rpy">
         <inertial>
-            <mass value="${m}" />
-            <origin xyz="${o_xyz}" rpy="${o_rpy}" />
-            <inertial ixx="${(m/12) * (y*y + z*z)}" ixy="0" ixz="0"
-                      iyy="${(m/12) * (x*x + z*z)}" iyz="0"
-                      izz="${(m/12) * (x*x + y*y)}" />
+            <mass value="${m}"/>
+            <origin xyz="${o_xyz}" rpy="${o_rpy}"/>
+            <inertia ixx="${(m/12) * (y*y + z*z)}" ixy="0" ixz="0"
+                     iyy="${(m/12) * (x*x + z*z)}" iyz="0"
+                     izz="${(m/12) * (x*x + y*y)}"/>
         </inertial>
     </xacro:macro>

File: ros2_ws/src/my_robot_description/urdf/mobile_base.xacro (robot description, xacro)
@@ -15,6 +15,6 @@
             <material name="blue" />
         </visual>
-        <xacro:box_intertia m="5.0" x="${base_length}" y="${base_width}" z="${base_height}"
-                            o_xyz="0 0 ${base_height / 2.0}" o_rpy="0 0 0" />
+        <xacro:box_inertia m="5.0" x="${base_length}" y="${base_width}" z="${base_height}"
+                           o_xyz="0 0 ${base_height / 2.0}" o_rpy="0 0 0" />
     </link>
     <xacro:macro name="wheel_link" params="prefix">

Commit message: robot arm project: arm base

File: ros2_ws/src/my_robot_description/urdf/common_properties.xacro (robot description, xacro)
@@ -6,4 +6,7 @@
     <material name="grey">
         <color rgba="0.5 0.5 0.5 1" />
+    </material>
+    <material name="orange">
+        <color rgba="1.0 0.5 0 1" />
     </material>
     <xacro:macro name="box_inertia" params="m x y z o_xyz o_rpy">
