Commit message: robot arm project: add arm and hand

File: ros2_ws/src/my_robot_description/urdf/arm.xacro (robot description, xacro)
@@ -1,7 +1,11 @@
 <?xml version="1.0"?>
-<robot name="arm" xmlns:xacro="http://www.ros.org/wiki/xacro">
+<robot xmlns:xacro="http://www.ros.org/wiki/xacro">
     <xacro:property name="arm_base_length" value="0.1" />
     <xacro:property name="arm_base_width" value="0.1" />
     <xacro:property name="arm_base_height" value ="0.02" />
+    <xacro:property name="forearm_radius" value="0.02" />
+    <xacro:property name="forearm_length" value="0.3" />
+    <xacro:property name="hand_radius" value="0.02" />
+    <xacro:property name="hand_length" value="0.3" />
     <link name="arm_base_link">
         <visual>
@@ -13,3 +17,36 @@
         </visual>
     </link>
+    <link name="forearm_link">
+        <visual>
+            <geometry>
+                <cylinder radius="${forearm_radius}" length="${forearm_length}" />
+            </geometry>
+            <origin xyz="0 0 ${forearm_length/2}" rpy="0 0 0" />
+            <material name="yellow" />
+        </visual>
+    </link>
+    <link name="hand_link">
+        <visual>
+            <geometry>
+                <cylinder radius="${hand_radius}" length="${hand_length}" />
+            </geometry>
+            <origin xyz="0 0 ${hand_length/2}" rpy="0 0 0" />
+            <material name="orange" />
+        </visual>
+    </link>
+    <!-- Joint -->
+    <joint name="arm_base_forearm_joint" type="revolute">
+        <parent link="arm_base_link" />
+        <child link="forearm_link" />
+        <origin xyz="0 0 ${arm_base_height}" rpy="0 0 0" />
+        <axis xyz="0 1 0" />
+        <limit lower="0" upper="${pi/2}" effort="100" velocity="100" />
+    </joint>
+    <joint name="forearm_hand_joint" type="revolute">
+        <parent link="forearm_link" />
+        <child link="hand_link" />
+        <origin xyz="0 0 ${forearm_length}" rpy="0 0 0" />
+        <axis xyz="0 1 0" />
+        <limit lower="0" upper="${pi/2}" effort="100" velocity="100" />
+    </joint>
 </robot>

File: ros2_ws/src/my_robot_description/urdf/common_properties.xacro (robot description, xacro)
@@ -9,4 +9,7 @@
     <material name="orange">
         <color rgba="1.0 0.5 0 1" />
+    </material>
+    <material name="yellow">
+        <color rgba="1.0 1.0 0 1" />
     </material>
     <xacro:macro name="box_inertia" params="m x y z o_xyz o_rpy">

Commit message: Adapt trobot for gazebo and add gazebo plugins

File: ros2_ws/src/my_robot_description/urdf/arm.xacro (robot description, xacro)
@@ -3,5 +3,5 @@
     <xacro:property name="arm_base_length" value="0.1" />
     <xacro:property name="arm_base_width" value="0.1" />
-    <xacro:property name="arm_base_height" value ="0.02" />
+    <xacro:property name="arm_base_height" value ="0.03" />
     <xacro:property name="forearm_radius" value="0.02" />
     <xacro:property name="forearm_length" value="0.3" />
@@ -13,7 +13,15 @@
                 <box size="${arm_base_length} ${arm_base_width} ${arm_base_height}" />
             </geometry>
-            <origin xyz="0 0 0" rpy="0 0 0" />
+            <origin xyz="0 0 ${arm_base_height / 2.0}" rpy="0 0 0" />
             <material name="orange" />
         </visual>
+        <collision>
+        <geometry>
+            <box size="${arm_base_length} ${arm_base_width} ${arm_base_height}" />
+            </geometry>
+            <origin xyz="0 0 ${arm_base_height / 2.0}" rpy="0 0 0" />
+        </collision>
+        <xacro:box_inertia m="5.0" x="${arm_base_length}" y="${arm_base_width}" z="${arm_base_height}"
+                           o_xyz="0 0 ${arm_base_height / 2.0}" o_rpy="0 0 0" />
     </link>
     <link name="forearm_link">
@@ -25,4 +33,12 @@
             <material name="yellow" />
         </visual>
+        <collision>
+            <geometry>
+                <cylinder radius="${forearm_radius}" length="${forearm_length}" />
+            </geometry>
+            <origin xyz="0 0 ${forearm_length/2}" rpy="0 0 0" />
+        </collision>
+        <xacro:cylinder_inertia m="0.3" r="${forearm_radius}" l="${forearm_length}"
+                                o_xyz="0 0 ${forearm_length / 2.0}" o_rpy="0 0 0" />
     </link>
     <link name="hand_link">
@@ -34,4 +50,12 @@
             <material name="orange" />
         </visual>
+        <collision>
+            <geometry>
+                <cylinder radius="${hand_radius}" length="${hand_length}" />
+            </geometry>
+            <origin xyz="0 0 ${hand_length/2}" rpy="0 0 0" />
+        </collision>
+        <xacro:cylinder_inertia m="0.3" r="${hand_radius}" l="${hand_length}"
+                                o_xyz="0 0 ${hand_length / 2.0}" o_rpy="0 0 0" />
     </link>
     <!-- Joint -->
@@ -42,4 +66,5 @@
         <axis xyz="0 1 0" />
         <limit lower="0" upper="${pi/2}" effort="100" velocity="100" />
+        <dynamics friction="0.3" damping="0.3" />
     </joint>
     <joint name="forearm_hand_joint" type="revolute">
@@ -49,4 +74,6 @@
         <axis xyz="0 1 0" />
         <limit lower="0" upper="${pi/2}" effort="100" velocity="100" />
+        <dynamics friction="0.3" damping="0.3" />
     </joint>
+    <!-- Gazebo -->
 </robot>

File: ros2_ws/src/my_robot_description/urdf/standalone_arm.urdf.xacro (robot description, xacro)
@@ -3,3 +3,4 @@
     <xacro:include filename="common_properties.xacro" />
     <xacro:include filename="arm.xacro" />
+    <xacro:include filename="arm_gazebo.xacro" />
 </robot>
